File: CPU.kicad_sch (KiCad schematic)
At the start: 75 parts, among them P4 DIN5, P5 DB9, Q1 2SC1815, Q2 2SC1959, U13 74LS08, Y1 14.31818 MHz

Commit message: Add files via upload
Updated to final versions.
Parts:
- added C201: 0.1uF, Capacitor_THT:C_Disc_D4.3mm_W1.9mm_P5.00mm, symbol Device:C
- added H9: MountingHole, MountingHole:MountingHole_3.2mm_M3_DIN965_Pad, symbol Mechanical:MountingHole_Pad
- added J201: Chroma Disconnect, Connector_PinHeader_2.54mm:PinHeader_2x01_P2.54mm_Vertical, symbol Connector:Conn_01x02_Male
- added J202: SVID_E, Connector_PinHeader_2.54mm:PinHeader_1x03_P2.54mm_Vertical, symbol Connector_Generic:Conn_01x03
- added R201: 75, Resistor_THT:R_Axial_DIN0207_L6.3mm_D2.5mm_P2.54mm_Vertical, symbol Device:R
- C4, C5, C6, C7: footprint Capacitor_THT:CP_Radial_D4.0mm_P1.50mm -> Capacitor_THT:CP_Radial_D5.0mm_P2.50mm
Connections:
- net BD4: now also UF8.5 (A3); no longer UF8.4 (A2)
- net BD5: now also UF8.4 (A2); no longer UF8.5 (A3)
- net CHROMA: now also C201.1, J201.2 (Pin_2); no longer FB8.2
- net GND: now also H9.1
- net VIDEO_OUT: now also J202.1 (Pin_1); no longer P4.5
- new net: J202.2 (Pin_2), P4.5
- new net: FB8.2, J201.1 (Pin_1)
- new net: C201.2, R201.1
- new net SVIDC: J202.3 (Pin_3), R201.2
Other:
- note added: "1-2: Normal 2-3: SVideo"
- note added: "Audio=WH Video=YL (Y) Chroma=RD (C)"
- note added: "Default: closed"
- note added: "S-Video Mod"
- moved on the sheet: C12, FB8, P4
