File: InpOutp.kicad_sch (KiCad schematic)
At the start: 41 parts, among them CN1 CONN_01X03, J301 Conn_02x12_Odd_Even, P1 MA156-12-2, P2 CASSETTE, P3 DIN6, P6 EXPANSION, P7 POWER TIP+, P8 CONN_01X20, SW1 Power

Commit message: Add files via upload
Updated to final versions.
Parts:
- removed F1: Polyfuse 0.25A, Fuse:Fuse_Littelfuse_395Series, symbol Device:Polyfuse_Small
Connections:
- net VCC: now also P8.4 (Pin_4)
Changed lines of the file:
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@@
   (title_block
     (title "VIC RELOADED")
-    (date "2022-05-14")
-    (rev "1.1-002D")
+    (date "2022-08-04")
+    (rev "1.1-002E")
     (company "Steve J. Gray and Rich Cini")
     (comment 1 "Transcribed from CBM VIC-20cr schematics 251027-01D")
@@
     (stroke (width 0) (type default) (color 0 0 0 0))
   )
-  (wire (pts (xy 104.775 49.53) (xy 136.525 49.53))
-    (stroke (width 0) (type default) (color 0 0 0 0))
-  )
   (wire (pts (xy 218.44 66.675) (xy 194.31 66.675))
     (stroke (width 0) (type default) (color 0 0 0 0))
@@
     (stroke (width 0) (type default) (color 0 0 0 0))
   )
-  (wire (pts (xy 117.475 31.75) (xy 104.775 31.75))
-    (stroke (width 0) (type default) (color 0 0 0 0))
-  )
   (wire (pts (xy 379.73 22.225) (xy 374.65 22.225))
     (stroke (width 0) (type default) (color 0 0 0 0))
@@
     (stroke (width 0) (type default) (color 0 0 0 0))
   )
-  (wire (pts (xy 104.775 31.75) (xy 104.775 49.53))
-    (stroke (width 0) (type default) (color 0 0 0 0))
-  )
   (wire (pts (xy 210.185 160.02) (xy 207.645 160.02))
     (stroke (width 0) (type default) (color 0 0 0 0))
@@
     (pin "1")
   )
-  (symbol (lib_id "power:VCC") (at 122.555 31.75 270) (unit 1)
-    (in_bom yes) (on_board yes)
-    (property "Reference" "#PWR0125" (id 0) (at 118.745 31.75 0)
-      (effects (font (size 1.27 1.27)) hide)
-    )
-    (property "Value" "VCC" (id 1) (at 125.7808 32.131 90)
-      (effects (font (size 1.27 1.27)) (justify left))
-    )
-    (property "Footprint" "" (id 2) (at 122.555 31.75 0)
-      (effects (font (size 1.27 1.27)) hide)
-    )
-    (property "Datasheet" "" (id 3) (at 122.555 31.75 0)
-      (effects (font (size 1.27 1.27)) hide)
-    )
-    (pin "1")
-  )
   (symbol (lib_id "power:VCC") (at 120.015 175.895 0) (mirror y) (unit 1)
     (in_bom yes) (on_board yes)
@@
     (pin "1")
   )
+  (symbol (lib_id "power:VCC") (at 136.525 49.53 90) (unit 1)
+    (in_bom yes) (on_board yes)
+    (property "Reference" "#PWR?" (id 0) (at 140.335 49.53 0)
+      (effects (font (size 1.27 1.27)) hide)
+    )
+    (property "Value" "VCC" (id 1) (at 133.2992 49.149 90)
+      (effects (font (size 1.27 1.27)) (justify left))
+    )
+    (property "Footprint" "" (id 2) (at 136.525 49.53 0)
+      (effects (font (size 1.27 1.27)) hide)
+    )
+    (property "Datasheet" "" (id 3) (at 136.525 49.53 0)
+      (effects (font (size 1.27 1.27)) hide)
+    )
+    (pin "1")
+  )
   (symbol (lib_id "power:GND") (at 160.655 246.38 0) (mirror y) (unit 1)
     (in_bom yes) (on_board yes)
@@
     (pin "9")
   )
-  (symbol (lib_id "Device:Polyfuse_Small") (at 120.015 31.75 90) (unit 1)
-    (in_bom yes) (on_board yes) (fields_autoplaced)
-    (property "Reference" "F1" (id 0) (at 120.015 27.1612 90))
-    (property "Value" "Polyfuse 0.25A" (id 1) (at 120.015 29.6981 90))
-    (property "Footprint" "Fuse:Fuse_Littelfuse_395Series" (id 2) (at 125.095 30.48 0)
-      (effects (font (size 1.27 1.27)) (justify left) hide)
-    )
-    (property "Datasheet" "~" (id 3) (at 120.015 31.75 0)
-      (effects (font (size 1.27 1.27)) hide)
-    )
-    (pin "1")
-    (pin "2")
-  )
 )
