File: VIC20Reloaded-1.1-002.kicad_pcb (KiCad board)
At the start: 2 copper layers, 254 x 136.6 mm, 136 parts, among them CN1 CONN_01X03, J301 Conn_02x12_Odd_Even, P1 MA156-12-2, P2 CASSETTE, P3 DIN6, P4 DIN5, P5 DB9, P6 EXPANSION, P7 POWER TIP+, P8 CONN_01X20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

Commit message: Add files via upload
Updated to final versions.
Parts:
- removed F1: Polyfuse 0.25A, Fuse:Fuse_Littelfuse_395Series
- added C201: 0.1uF, Capacitor_THT:C_Disc_D4.3mm_W1.9mm_P5.00mm, F.Cu at (214.6, 51.4)
- added H9: MountingHole, MountingHole:MountingHole_3.2mm_M3_DIN965_Pad, F.Cu at (177.5, 153.9)
- added J201: Chroma Disconnect, Connector_PinHeader_2.54mm:PinHeader_2x01_P2.54mm_Vertical, F.Cu at (211.1, 48.4)
- added J202: SVID_E, Connector_PinHeader_2.54mm:PinHeader_1x03_P2.54mm_Vertical, F.Cu at (133.7, 49.8)
- added R201: 75, Resistor_THT:R_Axial_DIN0207_L6.3mm_D2.5mm_P2.54mm_Vertical, F.Cu at (207.1, 50.9)
- C4, C5, C6, C7: footprint Capacitor_THT:CP_Radial_D4.0mm_P1.50mm -> Capacitor_THT:CP_Radial_D5.0mm_P2.50mm
- moved F2 8.33 mm to (281.2, 61.2), turned to 0 degrees
- moved R15 8.25 mm to (174.1, 146.9)
- moved C33 6.35 mm to (255.0, 58.0), turned to 90 degrees
- moved H4 6.27 mm to (290.4, 31.5)
- moved UC3 2.54 mm to (189.1, 125.3)
- moved UC2 2.54 mm to (174.1, 125.3)
- moved C31 1.16 mm to (263.9, 70.2)
- moved C32 1.16 mm to (263.9, 82.8)
- moved L3 1.16 mm to (268.0, 71.2)
- moved C4 1.14 mm to (177.4, 47.2)
- moved P6 1.12 mm to (133.3, 29.1)
- moved P4 0.94 mm to (104.1, 30.9)
- moved C5 0.53 mm to (222.0, 47.9)
- moved C48 0.51 mm to (211.1, 63.7)
- moved H2 0.51 mm to (52.5, 153.9)
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Connections:
- FB8 pad 2: CHROMA -> Net-(FB8-Pad2)
- P4 pad 5: VIDEO_OUT -> Net-(J202-Pad2)
- P8 pad 4: Net-(F1-Pad1) -> VCC
- UF8 pad 4: BD4 -> BD5
- UF8 pad 5: BD5 -> BD4
Routing:
- net SVIDC: track 0.00 -> 77.4 mm
- net VCC: track 1097.9 -> 1022.9 mm
- net A1: track 470.1 -> 397.3 mm
- net D5: track 193.5 -> 261.3 mm, vias 1 -> 0
- net Net-(F1-Pad1): track 51.7 -> 0.00 mm
- net JOY0: track 385.0 -> 334.8 mm, vias 1 -> 0
- net CPU_02: track 109.2 -> 154.6 mm
- net S01: track 128.0 -> 170.3 mm
- net R#W: track 369.7 -> 328.0 mm
- net GND: track 1477.7 -> 1519.1 mm
- net A3: track 423.7 -> 383.4 mm
- net CS_RAM1: track 130.7 -> 169.1 mm, vias 1 -> 0
- net D7: track 181.2 -> 219.0 mm
- net BD6: track 335.8 -> 373.0 mm, vias 4 -> 0
- net A9: track 255.4 -> 218.6 mm
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Other:
- board text added: "+ -"
- board text added: "Cr"
- board text added: "J201 Chroma Disconnect Default: in"
- board text added: "P4 Default 1-2"
- board text added: "Pin4"
- board text added: "Pin5"
- board text added: "VIC20RL-1.1-002E 080322"
- board text removed: "VIC20RL-1.1-002D 051422"
